File: bioelectric_cell_reprogramming/ion_concentration_biomodulator/EDA_designs/ion-concentration-biomodulator.kicad_pcb (KiCad board)
At the start: 4 copper layers, 90 x 78 mm, 37 parts, among them J1 532610671, J10 39-53-2045, J11 Conn_01x14_Pin, J12 Conn_01x14_Pin, J13 39-53-2045, J14 39-53-2045, J15 Conn_ARM_SWD_TagConnect_TC2030, J16 Conn_01x02_Socket, J18 EJ508A, J2 532610671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

Commit message: pushing v6
Parts:
- removed C2: 100nF, Capacitor_SMD:C_0402_1005Metric
- removed PE1: PeltierElement, Connector_PinSocket_2.54mm:PinSocket_1x02_P2.54mm_Vertical
- removed U6: STM32F410C8Tx, Package_QFP:LQFP-48_7x7mm_P0.5mm
- added C3: 100nF, Capacitor_SMD:C_0402_1005Metric, F.Cu at (173.8, 73.2)
- added J17: Conn_01x02_Pin, Connector_PinHeader_2.00mm:PinHeader_1x02_P2.00mm_Vertical, F.Cu at (134.8, 82.5)
- added J6: Conn_01x02_Pin, Connector_PinHeader_2.00mm:PinHeader_1x02_P2.00mm_Vertical, F.Cu at (135.0, 86.5)
- added J7: 6620XX11122_66200211122, peltier_cooler_socket_footprint:66200211122, F.Cu at (163.2, 56.2)
- added J9: IPL1-102-01-L-S-K, solenoid_footprint:CONN_IPL1-102-01-L-S-K_SAI, F.Cu at (149.7, 69.5)
- added Q2: NDT3055L, Package_TO_SOT_SMD:SOT-223-3_TabPin2, F.Cu at (121.4, 93.9)
- added Q4: NDT3055L, Package_TO_SOT_SMD:SOT-223-3_TabPin2, F.Cu at (121.4, 102.2)
- added Q5: NDT3055L, Package_TO_SOT_SMD:SOT-223-3_TabPin2, F.Cu at (121.4, 110.5)
- added Q6: NDT3055L, Package_TO_SOT_SMD:SOT-223-3_TabPin2, F.Cu at (121.5, 118.2)
- added U1: STM32F410CBTx, Package_QFP:LQFP-48_7x7mm_P0.5mm, F.Cu at (148.5, 101.2)
- J16: value Conn_01x02_Socket -> IPL1-104-01-L-D-K; footprint Connector_PinSocket_2.54mm:PinSocket_1x02_P2.54mm_Vertical -> pinch_solenoid:CONN_IPL1-104-01-x-D-x_SAI
- J5: value Conn_01x04_Socket -> S4B-PH-SM4-TB; footprint Connector_PinSocket_2.54mm:PinSocket_1x04_P2.54mm_Vertical -> co2_dev_board_male_socket:CONN4_S4B-PH-SM4-TB_JST
- U2, U3: footprint lm1084IT_regulator:T03B -> LDO_5V:T03B
- moved J16 47.0 mm to (120.0, 83.2), turned to 90 degrees
- moved G*** 7.02 mm to (186.5, 73.5)
- moved Q3 5.20 mm to (162.8, 62.5), turned to 180 degrees
- moved C23 3.48 mm to (154.2, 97.2)
- moved J5 0.93 mm to (168.7, 73.3)
Connections:
- J15 pad 3: unconnected-(J15-~{RESET}-Pad3) -> Net-(J15-~{RESET})
- J15 pad 6: unconnected-(J15-SWO-Pad6) -> Net-(J15-SWO)
- J16 pad 1: Net-(J16-Pin_1) -> Net-(Q2-D)
- J5 pad 1: GND -> /I2C_SCK
- J5 pad 2: /I2C_SCK -> GND
- J5 pad 3: /I2C_SDA -> +3.3V
- J5 pad 4: +3.3V -> /I2C_SDA
- Q1 pad 2: Net-(J16-Pin_1) -> Net-(Q1-D)
Routing:
- net Net-(Q6-D): track 0.00 -> 54.1 mm
- net Net-(Q5-D): track 0.00 -> 49.9 mm
- net /SOL1: track 0.00 -> 42.1 mm, vias 0 -> 2
- net /SOL3: track 0.00 -> 37.4 mm, vias 0 -> 2
- net /SOL4: track 0.00 -> 36.6 mm, vias 0 -> 2
- net /SWO: track 0.00 -> 35.5 mm, vias 0 -> 1
- net Net-(Q4-D): track 0.00 -> 32.5 mm
- net /SOL2: track 0.00 -> 31.9 mm, vias 0 -> 2
- net Net-(J15-SWO): track 0.00 -> 31.1 mm, vias 0 -> 1
- net Net-(J15-~{RESET}): track 0.00 -> 20.0 mm, vias 0 -> 1
- net Net-(Q2-D): track 0.00 -> 18.8 mm
- net Net-(Q1-D): track 0.00 -> 17.6 mm
- net Net-(J16-Pin_1): track 10.8 -> 0.00 mm
- net +3.3V: track 53.3 -> 63.6 mm, vias 14 -> 13
- net /NRST: track 20.9 -> 30.4 mm
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Other:
- board size 90 x 78 mm -> 98.5 x 78 mm
- board text added: "8/11/24 | Rev. 6"
- board text added: "barrel jack"
- board text added: "co2"
- board text added: "flow sensor array"
- board text added: "highdriver"
- board text added: "ldo 3.3"
- board text added: "ldo 5.0"
- board text added: "mp6 array"
- board text added: "pelt"
- board text added: "pinch sol"
- board text added: "pullups"
- board text added: "rst"
- board text added: "sol"
- board text added: "stm"
- board text added: "swo"
- board text removed: "8/11/24 | Rev. 5"

Commit message: pushing v7
Parts:
- D2: footprint LED_THT:LED_D3.0mm -> LED_THT:LED_D1.8mm_W1.8mm_H2.4mm_Horizontal_O3.81mm_Z1.6mm
- R1, R3: footprint Resistor_THT:R_Axial_DIN0207_L6.3mm_D2.5mm_P7.62mm_Horizontal -> Resistor_SMD:R_01005_0402Metric
- R2: footprint Resistor_THT:R_Axial_DIN0204_L3.6mm_D1.6mm_P5.08mm_Horizontal -> Resistor_SMD:R_01005_0402Metric
- moved C3 12.0 mm to (161.8, 73.8)
- moved C1 9.22 mm to (143.7, 67.1), turned to 0 degrees
- moved R2 5.07 mm to (149.5, 91.8), turned to 90 degrees
- moved G*** 4.26 mm to (182.2, 73.8)
- moved D2 2.41 mm to (146.8, 90.2), turned to -90 degrees
- moved J18 1.64 mm to (140.8, 62.5), turned to 180 degrees
- moved C21 1.55 mm to (147.3, 95.0), turned to 90 degrees
- moved C16 1.36 mm to (151.5, 107.0), turned to 180 degrees
- moved C23 0.35 mm to (154.0, 97.5)
Routing:
- net +3.3V: track 63.6 -> 72.9 mm, vias 13 -> 15
- net /I2C_SCK: track 133.3 -> 140.8 mm, vias 0 -> 2
- net GND: track 43.5 -> 36.5 mm, vias 23 -> 25
- net /I2C_SDA: track 169.7 -> 174.6 mm
- net /SOL4: track 36.6 -> 35.0 mm
- net /SOLEN_OUT: track 43.1 -> 44.3 mm
- net Net-(D2-A): track 2.29 -> 3.35 mm
Other:
- board text added: "8/13/24 | Rev. 7"
- board text removed: "8/11/24 | Rev. 6"
