File: bioelectric_cell_reprogramming/ion_concentration_biomodulator/EDA_designs/ion-concentration-biomodulator.kicad_sch (KiCad schematic)
At the start: 48 parts, among them J1 532610671, J10 39-53-2045, J11 Conn_01x14_Pin, J12 Conn_01x14_Pin, J13 39-53-2045, J14 39-53-2045, J15 Conn_ARM_SWD_TagConnect_TC2030, J16 IPL1-104-01-L-D-K, J17 Conn_01x02_Pin, J18 EJ508A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

Commit message: V7 fix: Increased area to add mounting holes and pushed receptacles to the edge of board
Parts:
- added H1, H2, H3, H4: MountingHole, MountingHole:MountingHole_2.2mm_M2, symbol Mechanical:MountingHole
