File: bioelectric_cell_reprogramming/AC_EF_testbed/EDA_designs/AC_EF.kicad_sch (KiCad schematic)
At the start: 10 parts, among them U1 STM32G431CBU3

Commit message: creating legacy branch before project restructure
Parts:
- added C10, C9: 100n, Capacitor_SMD:C_0402_1005Metric, symbol Device:C
- added C11: 1u, Capacitor_SMD:C_0402_1005Metric, symbol Device:C
- added C12, C13: 30p, symbol Device:C
- added C14, C15: 22u, symbol Device:C
- added D1: LED, symbol Device:LED
- added F1: 500mA, Fuse:Fuse_0603_1608Metric, symbol Device:Fuse
- added IC1: LTC3896EFE#PBF, SOP50P640X120-39N, symbol LTC3896EFE#PBF:LTC3896EFE#PBF
- added J1: USB_C_Receptacle_USB2.0_14P, Connector_USB:USB_C_Receptacle_GCT_USB4105-xx-A_16P_TopMnt_Horizontal, symbol Connector:USB_C_Receptacle_USB2.0_14P
- added J2: Conn_01x02_Socket, symbol Connector:Conn_01x02_Socket
- added J3: Conn_ARM_SWD_TagConnect_TC2030-NL, Connector:Tag-Connect_TC2030-IDC-NL_2x03_P1.27mm_Vertical, symbol Connector:Conn_ARM_SWD_TagConnect_TC2030-NL
- added R1: 10k, symbol Device:R
- added R2, R3: 5.1k, Resistor_SMD:R_0603_1608Metric, symbol Device:R
- added R4: 1k, symbol Device:R
- added SW1: SW_Push, Button_Switch_THT:SW_PUSH-12mm_Wuerth-430476085716, symbol Switch:SW_Push
- added SW2: SW_SPDT, symbol Switch:SW_SPDT
- added U2: USBLC6-2SC6, Package_TO_SOT_SMD:SOT-23-6, symbol Power_Protection:USBLC6-2SC6
- added U3: AMS1117-3.3, Package_TO_SOT_SMD:SOT-223-3_TabPin2, symbol Regulator_Linear:AMS1117-3.3
- added Y1: 16Mhz, symbol Device:Crystal_GND24
Connections:
- net +3.3V: now also C15.1, D1.2 (A), J3.1 (VCC), SW2.3 (C), U3.2 (VO)
- net GND: now also C10.2, C11.2, C12.2, C13.2, C14.2, C15.2, C9.2, J1.A1 (GND), J1.A12 (GND), J1.B1 (GND), J1.B12 (GND), J1.S1 (SHIELD), J2.2 (Pin_2), J3.5 (GND), R2.2, R3.2, R4.2, SW1.1, SW2.1 (A), U2.2 (GND), U3.1 (GND)
- net VREF: now reaches U1.20 (VREF+)
- net VREF: now also C10.1, C11.1
- net USB_D-: now reaches U1.33 (PA11)
- net USB_D-: now also U2.6 (I/O1)
- net USB_D+: now reaches U1.34 (PA12)
- net USB_D+: now also U2.4 (I/O2)
- net SWDIO: now reaches U1.36 (PA13)
- net SWDIO: now also J3.2 (SWDIO)
- net SWCLK: now reaches U1.37 (PA14)
- net SWCLK: now also J3.4 (SWCLK)
- net SWO: now reaches U1.41 (PB3)
- net SWO: now also J3.6 (SWO)
- net BOOT0: now reaches U1.46 (PB8)
- net BOOT0: now also R1.2
- net HSE_IN: now reaches U1.5 (PF0)
- net HSE_IN: now also C12.1, Y1.1
- net HSE_OUT: now reaches U1.6 (PF1)
- net HSE_OUT: now also C13.1, Y1.3
- net NRST: now reaches U1.7 (PG10)
- net NRST: now also C9.1, J3.3 (~{RESET}), SW1.2
- new net: F1.1, J1.A4 (VBUS), J1.A9 (VBUS), J1.B4 (VBUS), J1.B9 (VBUS)
- new net: J1.A5 (CC1), R2.1
- new net: J1.A6 (D+), J1.B6 (D+), U2.3 (I/O2)
- new net: J1.A7 (D-), J1.B7 (D-), U2.1 (I/O1)
- new net: J1.B5 (CC2), R3.1
- new net: R1.1, SW2.2 (B)
- new net: Y1.2, Y1.4
- new net +5V: C14.1, F1.2, U2.5 (VBUS), U3.3 (VI)
- new net +60V: J2.1 (Pin_1)
- new net PWR_LED_K: D1.1 (K), R4.1
Other:
- added sheet DCDC_inverter (DCDC_inverter.kicad_sch)
- moved on the sheet: C1, C2, C3, C4, C5, C6, C7, C8, FB1, U1
