File: bioelectric_cell_reprogramming/AC_EF_testbed/EDA_designs/DCDC_inverter.kicad_sch (KiCad schematic)
At the start: 11 parts, among them IC2 LTC3896EFE#PBF, Q1 IPD320N20N3GATMA1

Commit message: saving before merge
Parts:
- added C24, C25, C26, C27, C28: 0.1u, symbol Device:C
- added R6: 301k, symbol Device:R
Connections:
- net +60V: now also C24.1, C25.1, C26.1
- net -60V: now reaches IC2.1 (OVLO)
- net -60V: now also C20.1, C21.1, C22.1, C23.1, IC2.10 (VOUT-_2), IC2.15 (VOUT-_3), IC2.17 (FREQ), IC2.32 (EXTVCC), IC2.9 (VOUT-_1), C27.2, C28.2
- net at IC2.18 (DRVSET): now also IC2.19 (DRVUV), IC2.38 (INTVCC), IC2.8 (MODE), C28.1, R6.1
- net at IC2.5 (SS): now also C27.1, R6.2
- net at C16.2: now also C24.2, C25.2, C26.2
Other:
- moved on the sheet: C17, C18, C19, R5
