File: src/bioelectric_cell_reprogramming/acdc_stimulator/kicad/LTC6090_FB.kicad_sch (KiCad schematic)
At the start: 1 part, among them U4 LTC6090CFE-PBF

Commit message: ci: added error op amp to ADC
Parts:
- renumbered U4 to U1
Changed lines of the file:
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@@
 		(dnp no)
 		(fields_autoplaced yes)
-		(property "Reference" "U4"
+		(property "Reference" "U1"
 			(at 133.35 63.5 0)
 			(effects
@@
 		(instances
 			(project "acdc_stimulator"
-				(path "/ec70e9f6-566f-44ea-8141-5580f51beca4/5802e87b-47f9-4308-a638-d428408ef5d8"
-					(reference "U4")
+				(path "/ec70e9f6-566f-44ea-8141-5580f51beca4/adb33657-b159-4fcc-a216-5a35a6d2483a"
+					(reference "U1")
 					(unit 1)
 				)

Commit message: CI: footprint assignment done
Parts:
- U1: footprint TSSOP-16_FE/BA_LIT -> LTC6090CFE_PBF:TSSOP-16_FE&slash_BA_LIT
Changed lines of the file:
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@@
 			)
 		)
-		(property "Footprint" "TSSOP-16_FE/BA_LIT"
+		(property "Footprint" "LTC6090CFE_PBF:TSSOP-16_FE&slash_BA_LIT"
 			(at 110.49 73.66 0)
 			(effects

Commit message: ci: STM32 layout done and schematic annotated
Parts:
- renumbered U1 to U6
Changed lines of the file:
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@@
 		(dnp no)
 		(fields_autoplaced yes)
-		(property "Reference" "U1"
+		(property "Reference" "U6"
 			(at 133.35 63.5 0)
 			(effects
@@
 			(project "acdc_stimulator"
 				(path "/ec70e9f6-566f-44ea-8141-5580f51beca4/adb33657-b159-4fcc-a216-5a35a6d2483a"
-					(reference "U1")
+					(reference "U6")
 					(unit 1)
 				)
