File: src/bioelectric_cell_reprogramming/acdc_stimulator/kicad/acdc_stimulator.kicad_pcb (KiCad board)
At the start: 4 copper layers, 144 parts, among them IC1 AD9833BRM-REEL7, IC2 AD5122BCPZ10-RL7, IC3 LTC3896EFE#PBF, IC4 LTC3637IMSE#PBF, IC5 LTC3637IMSE#PBF, IC6 LTC3637IMSE#PBF, J1 Screw_Terminal_01x02, J2 Conn_ARM_SWD_TagConnect_TC203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, J3 USB_C_Receptacle_USB2.0_14P, J4 S4B-PH-SM4-TB, J5 IPL1-102-01-L-S-K, J6 Screw_Terminal_01x02, J7 IPL1-102-01-L-S-K, J8 6620XX11122_66200211122, J9 6620XX11122_66200211122, Q1 BSZ096N10LS5ATMA1, Q10 BSZ096N10LS5ATMA1, Q11 BSZ096N10LS5ATMA1, Q2 NDT3055L, Q3 BSC520N15NS3G, Q4 BSC520N15NS3G, Q5 IPD320N20N3GATMA1, Q6 BSZ096N10LS5ATMA1, Q7 BSZ096N10LS5ATMA1, Q8 IPB320P10LMATMA1, Q9 IPB320P10LMATMA1, SW1 SW_Push, SW2 SW_SPDT, U1 STM32G473RCTx, U2 AMS1117-3.3, U3 USBLC6-2SC6, U4 LTC6090CFE-PBF, U5 LTC6090CFE-PBF, U7 DRV8873HPWPR, Y1 16Mhz

Commit message: CI: v1 routing complete
Parts:
- moved H4 206.1 mm to (204.0, 148.0)
- moved H3 180.0 mm to (204.0, 27.0)
- moved H2 123.9 mm to (77.0, 148.0)
- moved H1 46.0 mm to (77.0, 27.0)
- moved C50 0.23 mm to (103.4, 127.0)
- moved C51 0.23 mm to (101.4, 127.0)
Routing:
- net +12V: track 26.1 -> 199.0 mm
- net /THERM_FB: track 0.00 -> 83.6 mm, vias 0 -> 2
- net /INCUBATOR_PELT_OUT: track 0.00 -> 81.8 mm, vias 0 -> 2
- net -60V: track 66.2 -> 138.0 mm, vias 4 -> 10
- net +5V: track 127.9 -> 193.9 mm, vias 0 -> 4
- net /SOLEN_OUT: track 0.00 -> 59.0 mm, vias 0 -> 4
- net +60V: track 145.0 -> 202.6 mm, vias 0 -> 3
- net /VAC_ON: track 0.00 -> 56.9 mm, vias 0 -> 4
- net /H_Bridge_IN1: track 0.00 -> 54.8 mm, vias 0 -> 6
- net /I2C_SDA: track 4.14 -> 58.3 mm, vias 0 -> 2
- net /I2C_SCL: track 4.03 -> 55.9 mm, vias 0 -> 2
- net /H_BRIDGE_IN1: track 0.00 -> 49.0 mm, vias 0 -> 4
- net /H_BRIDGE_FAULT: track 0.00 -> 48.2 mm, vias 0 -> 4
- net /H_BRIDGE_IN2: track 0.00 -> 47.8 mm, vias 0 -> 4
- net /DAC_AC: track 0.00 -> 39.7 mm, vias 0 -> 2
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- added copper zone on In2.Cu, net +3.3V
- added copper zone on F.Cu, net /CO2 Solenoid
- added copper zone on F.Cu, net /pelt_cooler/OUT1
- added copper zone on F.Cu, net /pelt_cooler/OUT2
- added copper zone on In1.Cu, net GND
Other:
- board outline added: 139 x 133 mm

Commit message: ci: v1 routing complete
Routing:
- net Net-(J6-Pin_2): track 52.7 -> 52.0 mm
- net -60V: vias 10 -> 9

Commit message: ci: silkscreen cleaned up
Routing:
- net +3.3V: vias 58 -> 59
