File: src/bioelectric_cell_reprogramming/acdc_stimulator/kicad/acdc_stimulator.kicad_pcb (KiCad board)
At the start: 4 copper layers, 139 x 133 mm, 145 parts, among them IC1 AD9833BRM-REEL7, IC3 LTC3896EFE#PBF, IC4 LTC3637IMSE#PBF, IC5 LTC3637IMSE#PBF, IC6 LTC3637IMSE#PBF, IC7 AD5160BRJZ10-RL7, J1 Screw_Terminal_01x02, J2 Conn_ARM_SWD_TagConnect_TC203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, J3 USB_C_Receptacle_USB2.0_14P, J4 S4B-PH-SM4-TB, J5 IPL1-102-01-L-S-K, J6 Screw_Terminal_01x02, J7 IPL1-102-01-L-S-K, J8 6620XX11122_66200211122, J9 6620XX11122_66200211122, Q1 BSZ096N10LS5ATMA1, Q10 BSZ096N10LS5ATMA1, Q11 BSZ096N10LS5ATMA1, Q2 NDT3055L, Q3 BSC520N15NS3G, Q4 BSC520N15NS3G, Q5 IPD320N20N3GATMA1, Q6 BSZ096N10LS5ATMA1, Q7 BSZ096N10LS5ATMA1, Q8 IPB320P10LMATMA1, Q9 IPB320P10LMATMA1, SW1 SW_Push, SW2 SW_SPDT, U1 STM32G473RCTx, U2 AMS1117-3.3, U3 USBLC6-2SC6, U4 LTC6090CFE-PBF, U5 LTC6090CFE-PBF, U7 DRV8873HPWPR, Y1 16Mhz

Commit message: ci: manufacturing files generated
Routing:
- net +3.3V: track 46.9 -> 21.1 mm
- net +12V: track 201.7 -> 176.6 mm
- net +5V: track 207.0 -> 183.9 mm
- added copper zone on F.Cu, net +12V
Changed lines of the file:
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@@
 		(pad_to_mask_clearance 0)
 		(allow_soldermask_bridges_in_footprints no)
+		(aux_axis_origin 71 154)
+		(grid_origin 71 154)
 		(pcbplotparams
-			(layerselection 0x00010fc_ffffffff)
+			(layerselection 0x00010e8_ffffffff)
 			(plot_on_all_layers_selection 0x0000000_00000000)
 			(disableapertmacros no)
@@
 			(viasonmask no)
 			(mode 1)
-			(useauxorigin no)
+			(useauxorigin yes)
 			(hpglpennumber 1)
 			(hpglpenspeed 20)
@@
 			(psnegative no)
 			(psa4output no)
-			(plotreference yes)
-			(plotvalue yes)
-			(plotfptext yes)
+			(plotreference no)
+			(plotvalue no)
+			(plotfptext no)
 			(plotinvisibletext no)
 			(sketchpadsonfab no)
@@
 			(outputformat 1)
 			(mirror no)
-			(drillshape 1)
+			(drillshape 0)
 			(scaleselection 1)
-			(outputdirectory "")
+			(outputdirectory "./")
 		)
 	)
@@
 	)
 	(segment
-		(start 176.895 133.85)
-		(end 176.895 133.305)
-		(width 2)
-		(layer "F.Cu")
-		(net 4)
-	)
-	(segment
 		(start 182.275 145.475)
 		(end 88.912298 145.475)
@@
 	)
 	(segment
-		(start 185 125.2)
-		(end 185 126.375)
-		(width 2)
-		(layer "F.Cu")
-		(net 4)
-	)
-	(segment
 		(start 112.25 145.475)
 		(end 112.05 145.475)
@@
 	)
 	(segment
-		(start 185 126.375)
-		(end 193.4 134.775)
-		(width 2)
-		(layer "F.Cu")
-		(net 4)
-	)
-	(segment
 		(start 101.45 134.875)
 		(end 101.45 128.6)
@@
 	)
 	(segment
-		(start 176.895 133.305)
-		(end 185 125.2)
-		(width 2)
-		(layer "F.Cu")
-		(net 4)
-	)
-	(segment
 		(start 114.249999 143.475001)
 		(end 112.25 145.475)
@@
 	)
 	(segment
-		(start 176.995 86.5005)
-		(end 176.995 88.4)
-		(width 0.5)
-		(layer "F.Cu")
-		(net 9)
-	)
-	(segment
-		(start 184.7455 78.75)
-		(end 176.995 86.5005)
-		(width 0.5)
-		(layer "F.Cu")
-		(net 9)
-	)
-	(segment
-		(start 190.25 78.75)
-		(end 193.1 81.6)
-		(width 0.5)
-		(layer "F.Cu")
-		(net 9)
-	)
-	(segment
 		(start 148.29038 106.33462)
 		(end 166.225 88.4)
@@
 	)
 	(segment
-		(start 205.25 67.75)
-		(end 194.25 78.75)
-		(width 0.5)
-		(layer "F.Cu")
-		(net 9)
-	)
-	(segment
 		(start 196.0625 48.255)
 		(end 199.905 48.255)
@@
 	)
 	(segment
-		(start 205.25 53.6)
-		(end 205.25 67.75)
-		(width 0.5)
-		(layer "F.Cu")
-		(net 9)
-	)
-	(segment
 		(start 80.95 85.175)
 		(end 81.175 85.4)
@@
 	)
 	(segment
-		(start 194.25 78.75)
-		(end 190.25 78.75)
+		(start 205.25 67.75)
+		(end 193.1 79.9)
 		(width 0.5)
 		(layer "F.Cu")
@@
 	)
 	(segment
+		(start 205.25 53.6)
+		(end 205.25 67.75)
+		(width 0.5)
+		(layer "F.Cu")
+		(net 9)
+	)
+	(segment
 		(start 81.375 83.85)
 		(end 80.95 84.275)
@@
 	)
 	(segment
-		(start 96.35 92.2)
-		(end 96.35 102.65)
-		(width 0.3)
+		(start 193.1 79.9)
+		(end 193.1 88.325)
+		(width 0.5)
 		(layer "F.Cu")
 		(net 9)
 	)
 	(segment
-		(start 193.1 81.6)
-		(end 193.1 88.325)
-		(width 0.5)
+		(start 96.35 92.2)
+		(end 96.35 102.65)
+		(width 0.3)
 		(layer "F.Cu")
 		(net 9)
@@
 	)
 	(segment
-		(start 190.25 78.75)
-		(end 184.7455 78.75)
-		(width 0.5)
-		(layer "F.Cu")
-		(net 9)
-	)
-	(segment
 		(start 81.9125 83.85)
 		(end 81.375 83.85)
@@
 	)
 	(segment
-		(start 177.05 108.65)
-		(end 184.75 100.95)
-		(width 0.5)
-		(layer "F.Cu")
-		(net 10)
-	)
-	(segment
 		(start 102.75 86.225)
 		(end 102.75 85.4)
@@
 	)
 	(segment
-		(start 177.05 110.55)
-		(end 177.05 108.65)
-		(width 0.5)
-		(layer "F.Cu")
-		(net 10)
-	)
-	(segment
 		(start 99.325 91.035)
 		(end 100.161526 91.035)
@@
 	)
 	(segment
-		(start 184.75 100.95)
-		(end 193.1 109.3)
-		(width 0.5)
-		(layer "F.Cu")
-		(net 10)
-	)
-	(segment
 		(start 116.3 85.135)
 		(end 116.15 84.985)
@@
 	)
 	(segment
-		(start 193.1 109.3)
-		(end 193.1 110.525)
-		(width 0.5)
-		(layer "F.Cu")
-		(net 10)
-	)
-	(segment
 		(start 133.5125 101.5125)
 		(end 133.5125 102.6875)
@@
 	)
 	(zone
+		(net 10)
+		(net_name "+3.3V")
+		(layer "F.Cu")
+		(hatch edge 0.5)
+		(priority 13)
+		(connect_pads yes
+			(clearance 0.3)
+		)
+		(min_thickness 0.25)
+		(filled_areas_thickness no)
+		(fill yes
+			(thermal_gap 0.5)
+			(thermal_bridge_width 0.5)
+		)
+		(polygon
+			(pts
+				(xy 182.1 110.825) (xy 182.825 110.1) (xy 186.65 110.1) (xy 187.675 111.125) (xy 193.85 111.125)
+				(xy 194.05 110.925) (xy 194.05 101.275) (xy 191.85 99.075) (xy 178.15 99.075) (xy 176.725 100.5)
+				(xy 176.725 110.625) (xy 176.925 110.825)
+			)
+		)
+	)
+	(zone
 		(net 13)
 		(net_name "/DCDC_inverter/INTVCC")
@@
 	)
 	(zone
+		(net 4)
+		(net_name "+12V")
+		(layer "F.Cu")
+		(hatch edge 0.5)
+		(priority 14)
+		(connect_pads yes
+			(clearance 0.3)
+		)
+		(min_thickness 0.25)
+		(filled_areas_thickness no)
+		(fill yes
+			(thermal_gap 0.5)
+			(thermal_bridge_width 0.5)
+		)
+		(polygon
+			(pts
+				(xy 176.55 134.25) (xy 176.4 134.1) (xy 176.4 125.025) (xy 178.2 123.225) (xy 193.125 123.225) (xy 194.4 124.5)
+				(xy 194.4 135.225) (xy 191.275 138.35) (xy 188.075 138.35) (xy 187.1 137.375) (xy 187.1 134.6) (xy 186.75 134.25)
+			)
+		)
+	)
+	(zone
 		(net 2)
 		(net_name "GND")
@@
 			)
 		)
+	)
+	(zone
+		(net 9)
+		(net_name "+5V")
+		(layer "F.Cu")
+		(hatch edge 0.5)
+		(priority 13)
+		(connect_pads yes
+			(clearance 0.3)
+		)
+		(min_thickness 0.25)
+		(filled_areas_thickness no)
+		(fill yes
+			(thermal_gap 0.5)
+			(thermal_bridge_width 0.5)
+		)
+		(polygon
+			(pts
+				(xy 181.975 88.65) (xy 182.725 87.9) (xy 186.625 87.9) (xy 187.675 88.95) (xy 193.825 88.95) (xy 194.05 88.725)
+				(xy 194.05 79.1) (xy 191.85 76.9) (xy 178.15 76.9) (xy 176.725 78.325) (xy 176.725 88.45) (xy 176.925 88.65)
+			)
+		)
