File: src/bioelectric_cell_reprogramming/acdc_stimulator/kicad/H_Bridge.kicad_sch (KiCad schematic)
At the start: 8 parts, among them Q4 BSZ096N10LS5ATMA1, Q5 IPB320P10LMATMA1, Q6 BSZ096N10LS5ATMA1, Q7 IPB320P10LMATMA1, Q8 BSZ096N10LS5ATMA1, Q9 BSZ096N10LS5ATMA1

Commit message: CI: footprint assignment done
Parts:
- Q4, Q6, Q8, Q9: footprint BSZ060NE2LS -> BSZ096N10LS5ATMA1:BSZ060NE2LS
- Q5, Q7: footprint IPB320P10LMATMA1 -> IPB320P10LMATMA1:IPB320P10LMATMA1
- R13, R14: footprint (none) -> Resistor_SMD:R_0402_1005Metric
Changed lines of the file:
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@@
 			)
 		)
-		(property "Footprint" "BSZ060NE2LS"
+		(property "Footprint" "BSZ096N10LS5ATMA1:BSZ060NE2LS"
 			(at 110.49 218.11 0)
 			(effects
@@
 			)
 		)
-		(property "Footprint" ""
+		(property "Footprint" "Resistor_SMD:R_0402_1005Metric"
 			(at 102.362 80.01 90)
 			(effects
@@
 			)
 		)
-		(property "Footprint" "BSZ060NE2LS"
+		(property "Footprint" "BSZ096N10LS5ATMA1:BSZ060NE2LS"
 			(at 83.82 188.9 0)
 			(effects
@@
 			)
 		)
-		(property "Footprint" ""
+		(property "Footprint" "Resistor_SMD:R_0402_1005Metric"
 			(at 174.752 80.01 90)
 			(effects
@@
 			)
 		)
-		(property "Footprint" "BSZ060NE2LS"
+		(property "Footprint" "BSZ096N10LS5ATMA1:BSZ060NE2LS"
 			(at 171.45 219.38 0)
 			(effects
@@
 			)
 		)
-		(property "Footprint" "BSZ060NE2LS"
+		(property "Footprint" "BSZ096N10LS5ATMA1:BSZ060NE2LS"
 			(at 196.85 188.9 0)
 			(effects
@@
 			)
 		)
-		(property "Footprint" "IPB320P10LMATMA1"
+		(property "Footprint" "IPB320P10LMATMA1:IPB320P10LMATMA1"
 			(at 161.29 -9.83 0)
 			(effects
@@
 			)
 		)
-		(property "Footprint" "IPB320P10LMATMA1"
+		(property "Footprint" "IPB320P10LMATMA1:IPB320P10LMATMA1"
 			(at 120.65 -9.83 0)
 			(effects

Commit message: ci: STM32 layout done and schematic annotated
Parts:
- renumbered Q4 to Q10, Q9 to Q11, Q8 to Q6, Q6 to Q7, Q7 to Q8, Q5 to Q9, R13 to R22, R14 to R23
Changed lines of the file:
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@@
 		(dnp no)
 		(fields_autoplaced yes)
-		(property "Reference" "Q6"
+		(property "Reference" "Q7"
 			(at 101.6 115.57 0)
 			(effects
@@
 			(project "acdc_stimulator"
 				(path "/ec70e9f6-566f-44ea-8141-5580f51beca4/ea1d9750-8e7d-4025-a446-b33892bad04a"
-					(reference "Q6")
+					(reference "Q7")
 					(unit 1)
 				)
@@
 		(dnp no)
 		(fields_autoplaced yes)
-		(property "Reference" "R13"
+		(property "Reference" "R22"
 			(at 106.68 78.7399 0)
 			(effects
@@
 			(project ""
 				(path "/ec70e9f6-566f-44ea-8141-5580f51beca4/ea1d9750-8e7d-4025-a446-b33892bad04a"
-					(reference "R13")
+					(reference "R22")
 					(unit 1)
 				)
@@
 		(dnp no)
 		(fields_autoplaced yes)
-		(property "Reference" "#PWR045"
+		(property "Reference" "#PWR070"
 			(at 78.74 132.08 0)
 			(effects
@@
 			(project ""
 				(path "/ec70e9f6-566f-44ea-8141-5580f51beca4/ea1d9750-8e7d-4025-a446-b33892bad04a"
-					(reference "#PWR045")
+					(reference "#PWR070")
 					(unit 1)
 				)
@@
 		(dnp no)
 		(fields_autoplaced yes)
-		(property "Reference" "#PWR048"
+		(property "Reference" "#PWR072"
 			(at 228.6 102.87 0)
 			(effects
@@
 			(project "acdc_stimulator"
 				(path "/ec70e9f6-566f-44ea-8141-5580f51beca4/ea1d9750-8e7d-4025-a446-b33892bad04a"
-					(reference "#PWR048")
+					(reference "#PWR072")
 					(unit 1)
 				)
@@
 		(dnp no)
 		(fields_autoplaced yes)
-		(property "Reference" "Q8"
+		(property "Reference" "Q6"
 			(at 74.93 86.36 0)
 			(effects
@@
 			(project "acdc_stimulator"
 				(path "/ec70e9f6-566f-44ea-8141-5580f51beca4/ea1d9750-8e7d-4025-a446-b33892bad04a"
-					(reference "Q8")
+					(reference "Q6")
 					(unit 1)
 				)
@@
 		(dnp no)
 		(fields_autoplaced yes)
-		(property "Reference" "#PWR047"
+		(property "Reference" "#PWR069"
 			(at 52.07 102.87 0)
 			(effects
@@
 			(project "acdc_stimulator"
 				(path "/ec70e9f6-566f-44ea-8141-5580f51beca4/ea1d9750-8e7d-4025-a446-b33892bad04a"
-					(reference "#PWR047")
+					(reference "#PWR069")
 					(unit 1)
 				)
@@
 		(dnp no)
 		(fields_autoplaced yes)
-		(property "Reference" "#PWR046"
+		(property "Reference" "#PWR071"
 			(at 203.2 133.35 0)
 			(effects
@@
 			(project ""
 				(path "/ec70e9f6-566f-44ea-8141-5580f51beca4/ea1d9750-8e7d-4025-a446-b33892bad04a"
-					(reference "#PWR046")
+					(reference "#PWR071")
 					(unit 1)
 				)
@@
 		(dnp no)
 		(fields_autoplaced yes)
-		(property "Reference" "R14"
+		(property "Reference" "R23"
 			(at 179.07 78.7399 0)
 			(effects
@@
 			(project "acdc_stimulator"
 				(path "/ec70e9f6-566f-44ea-8141-5580f51beca4/ea1d9750-8e7d-4025-a446-b33892bad04a"
-					(reference "R14")
+					(reference "R23")
 					(unit 1)
 				)
@@
 		(dnp no)
 		(fields_autoplaced yes)
-		(property "Reference" "Q4"
+		(property "Reference" "Q10"
 			(at 180.34 116.84 0)
 			(effects
@@
 			(project ""
 				(path "/ec70e9f6-566f-44ea-8141-5580f51beca4/ea1d9750-8e7d-4025-a446-b33892bad04a"
-					(reference "Q4")
+					(reference "Q10")
 					(unit 1)
 				)
@@
 		(dnp no)
 		(fields_autoplaced yes)
-		(property "Reference" "Q9"
+		(property "Reference" "Q11"
 			(at 205.74 86.36 0)
 			(effects
@@
 			(project "acdc_stimulator"
 				(path "/ec70e9f6-566f-44ea-8141-5580f51beca4/ea1d9750-8e7d-4025-a446-b33892bad04a"
-					(reference "Q9")
+					(reference "Q11")
 					(unit 1)
 				)
@@
 		(on_board yes)
 		(dnp no)
-		(property "Reference" "Q5"
+		(property "Reference" "Q9"
 			(at 161.29 92.7101 0)
 			(effects
@@
 			(project ""
 				(path "/ec70e9f6-566f-44ea-8141-5580f51beca4/ea1d9750-8e7d-4025-a446-b33892bad04a"
-					(reference "Q5")
+					(reference "Q9")
 					(unit 1)
 				)
@@
 		(on_board yes)
 		(dnp no)
-		(property "Reference" "Q7"
+		(property "Reference" "Q8"
 			(at 120.65 90.1699 0)
 			(effects
@@
 			(project "acdc_stimulator"
 				(path "/ec70e9f6-566f-44ea-8141-5580f51beca4/ea1d9750-8e7d-4025-a446-b33892bad04a"
-					(reference "Q7")
+					(reference "Q8")
 					(unit 1)
 				)

Commit message: fixed some more clearance errors
Parts:
- R22, R23: Distributor Link (none) -> https://jlcpcb.com/partdetail/259901-NQ02WGJ0103TCE/C270371; Manufacturer (none) -> UNI-ROYAL(Uniroyal Elec); Manufacturer Part Number (none) -> NQ02WGJ0103TCE
Changed lines of the file:
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@@
+			)
+		)
+		(property "Distributor Link" ""
+			(at 88.9 123.19 0)
+			(effects
+				(font
+					(size 1.27 1.27)
+				)
+				(hide yes)
+			)
+		)
+		(property "Manufacturer" ""
+			(at 88.9 123.19 0)
+			(effects
+				(font
+					(size 1.27 1.27)
+				)
+				(hide yes)
+			)
+		)
+		(property "Manufacturer Part Number" ""
+			(at 88.9 123.19 0)
+			(effects
+				(font
+					(size 1.27 1.27)
+				)
+				(hide yes)
 			)
 		)
@@
 		)
 		(property "Description" "Resistor"
+			(at 104.14 80.01 0)
+			(effects
+				(font
+					(size 1.27 1.27)
+				)
+				(hide yes)
+			)
+		)
+		(property "Distributor Link" "https://jlcpcb.com/partdetail/259901-NQ02WGJ0103TCE/C270371"
+			(at 104.14 80.01 0)
+			(effects
+				(font
+					(size 1.27 1.27)
+				)
+				(hide yes)
+			)
+		)
+		(property "Manufacturer" "UNI-ROYAL(Uniroyal Elec)"
+			(at 104.14 80.01 0)
+			(effects
+				(font
+					(size 1.27 1.27)
+				)
+				(hide yes)
+			)
+		)
+		(property "Manufacturer Part Number" "NQ02WGJ0103TCE"
 			(at 104.14 80.01 0)
 			(effects
@@
 			)
 		)
+		(property "Distributor Link" ""
+			(at 62.23 93.98 0)
+			(effects
+				(font
+					(size 1.27 1.27)
+				)
+				(hide yes)
+			)
+		)
+		(property "Manufacturer" ""
+			(at 62.23 93.98 0)
+			(effects
+				(font
+					(size 1.27 1.27)
+				)
+				(hide yes)
+			)
+		)
+		(property "Manufacturer Part Number" ""
+			(at 62.23 93.98 0)
+			(effects
+				(font
+					(size 1.27 1.27)
+				)
+				(hide yes)
+			)
+		)
 		(pin "8"
 		)
@@
 		)
 		(property "Description" "Resistor"
+			(at 176.53 80.01 0)
+			(effects
+				(font
+					(size 1.27 1.27)
+				)
+				(hide yes)
+			)
+		)
+		(property "Distributor Link" "https://jlcpcb.com/partdetail/259901-NQ02WGJ0103TCE/C270371"
+			(at 176.53 80.01 0)
+			(effects
+				(font
+					(size 1.27 1.27)
+				)
+				(hide yes)
+			)
+		)
+		(property "Manufacturer" "UNI-ROYAL(Uniroyal Elec)"
+			(at 176.53 80.01 0)
+			(effects
+				(font
+					(size 1.27 1.27)
+				)
+				(hide yes)
+			)
+		)
+		(property "Manufacturer Part Number" "NQ02WGJ0103TCE"
 			(at 176.53 80.01 0)
 			(effects
@@
 			)
 		)
+		(property "Distributor Link" ""
+			(at 193.04 124.46 0)
+			(effects
+				(font
+					(size 1.27 1.27)
+				)
+				(hide yes)
+			)
+		)
+		(property "Manufacturer" ""
+			(at 193.04 124.46 0)
+			(effects
+				(font
+					(size 1.27 1.27)
+				)
+				(hide yes)
+			)
+		)
+		(property "Manufacturer Part Number" ""
+			(at 193.04 124.46 0)
+			(effects
+				(font
+					(size 1.27 1.27)
+				)
+				(hide yes)
+			)
+		)
 		(pin "8"
 		)
@@
 			)
 		)
+		(property "Distributor Link" ""
+			(at 218.44 93.98 0)
+			(effects
+				(font
+					(size 1.27 1.27)
+				)
+				(hide yes)
+			)
+		)
+		(property "Manufacturer" ""
+			(at 218.44 93.98 0)
+			(effects
+				(font
+					(size 1.27 1.27)
+				)
+				(hide yes)
+			)
+		)
+		(property "Manufacturer Part Number" ""
+			(at 218.44 93.98 0)
+			(effects
+				(font
+					(size 1.27 1.27)
+				)
+				(hide yes)
+			)
+		)
 		(pin "8"
 		)
@@
 				)
 				(justify left top)
+				(hide yes)
+			)
+		)
+		(property "Distributor Link" ""
+			(at 172.72 88.9 0)
+			(effects
+				(font
+					(size 1.27 1.27)
+				)
+				(hide yes)
+			)
+		)
+		(property "Manufacturer" ""
+			(at 172.72 88.9 0)
+			(effects
+				(font
+					(size 1.27 1.27)
+				)
+				(hide yes)
+			)
+		)
+		(property "Manufacturer Part Number" ""
+			(at 172.72 88.9 0)
+			(effects
+				(font
+					(size 1.27 1.27)
+				)
 				(hide yes)
 			)
@@
 				(hide yes)
 			)
+		)
+		(property "Distributor Link" ""
+			(at 109.22 88.9 0)
+			(effects
+				(font
+					(size 1.27 1.27)
+				)
+				(hide yes)
+			)
+		)
+		(property "Manufacturer" ""
+			(at 109.22 88.9 0)
+			(effects
+				(font
+					(size 1.27 1.27)
+				)
+				(hide yes)
+			)
+		)
+		(property "Manufacturer Part Number" ""
+			(at 109.22 88.9 0)
+			(effects
+				(font
+					(size 1.27 1.27)
+				)
+				(hide yes)
+			)

Commit message: BOM in progress
Parts:
- Q10, Q11, Q6, Q7: Distributor Link (none) -> https://www.mouser.com/ProductDetail/Infineon-Technologies/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; Manufacturer (none) -> Infineon Technologies; Manufacturer Part Number (none) -> BSZ096N10LS5ATMA1
- Q8, Q9: Distributor Link (none) -> https://jlcpcb.com/partdetail/3852120-IPB320P10LMATMA1/C328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; Manufacturer (none) -> Infineon Technologies; Manufacturer Part Number (none) -> C3289219
Changed lines of the file:
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@@
 			)
 		)
-		(property "Distributor Link" ""
+		(property "Distributor Link" "https://www.mouser.com/ProductDetail/Infineon-Technologies/BSZ096N10LS5ATMA1?qs=Qyx3PVvfm65D5XP%2FZXFciQ%3D%3D"
 			(at 88.9 123.19 0)
 			(effects
@@
 			)
 		)
-		(property "Manufacturer" ""
+		(property "Manufacturer" "Infineon Technologies "
 			(at 88.9 123.19 0)
 			(effects
@@
 			)
 		)
-		(property "Manufacturer Part Number" ""
+		(property "Manufacturer Part Number" "BSZ096N10LS5ATMA1"
+			(at 88.9 123.19 0)
+			(effects
+				(font
+					(size 1.27 1.27)
+				)
+				(hide yes)
+			)
+		)
+		(property "JLCPCB Part #" ""
 			(at 88.9 123.19 0)
 			(effects
@@
 		)
 		(property "Manufacturer Part Number" "NQ02WGJ0103TCE"
+			(at 104.14 80.01 0)
+			(effects
+				(font
+					(size 1.27 1.27)
+				)
+				(hide yes)
+			)
+		)
+		(property "JLCPCB Part #" ""
 			(at 104.14 80.01 0)
 			(effects
@@
 			)
 		)
-		(property "Distributor Link" ""
+		(property "Distributor Link" "https://www.mouser.com/ProductDetail/Infineon-Technologies/BSZ096N10LS5ATMA1?qs=Qyx3PVvfm65D5XP%2FZXFciQ%3D%3D"
 			(at 62.23 93.98 0)
 			(effects
@@
 			)
 		)
-		(property "Manufacturer" ""
+		(property "Manufacturer" "Infineon Technologies "
 			(at 62.23 93.98 0)
 			(effects
@@
 			)
 		)
-		(property "Manufacturer Part Number" ""
+		(property "Manufacturer Part Number" "BSZ096N10LS5ATMA1"
+			(at 62.23 93.98 0)
+			(effects
+				(font
+					(size 1.27 1.27)
+				)
+				(hide yes)
+			)
+		)
+		(property "JLCPCB Part #" ""
 			(at 62.23 93.98 0)
 			(effects
@@
 		)
 		(property "Manufacturer Part Number" "NQ02WGJ0103TCE"
+			(at 176.53 80.01 0)
+			(effects
+				(font
+					(size 1.27 1.27)
+				)
+				(hide yes)
+			)
+		)
+		(property "JLCPCB Part #" ""
 			(at 176.53 80.01 0)
 			(effects
@@
 			)
 		)
-		(property "Distributor Link" ""
+		(property "Distributor Link" "https://www.mouser.com/ProductDetail/Infineon-Technologies/BSZ096N10LS5ATMA1?qs=Qyx3PVvfm65D5XP%2FZXFciQ%3D%3D"
 			(at 193.04 124.46 0)
 			(effects
@@
 			)
 		)
-		(property "Manufacturer" ""
+		(property "Manufacturer" "Infineon Technologies "
 			(at 193.04 124.46 0)
 			(effects
@@
 			)
 		)
-		(property "Manufacturer Part Number" ""
+		(property "Manufacturer Part Number" "BSZ096N10LS5ATMA1"
+			(at 193.04 124.46 0)
+			(effects
+				(font
+					(size 1.27 1.27)
+				)
+				(hide yes)
+			)
+		)
+		(property "JLCPCB Part #" ""
 			(at 193.04 124.46 0)
 			(effects
@@
 			)
 		)
-		(property "Distributor Link" ""
+		(property "Distributor Link" "https://www.mouser.com/ProductDetail/Infineon-Technologies/BSZ096N10LS5ATMA1?qs=Qyx3PVvfm65D5XP%2FZXFciQ%3D%3D"
 			(at 218.44 93.98 0)
 			(effects
@@
 			)
 		)
-		(property "Manufacturer" ""
+		(property "Manufacturer" "Infineon Technologies "
 			(at 218.44 93.98 0)
 			(effects
@@
 			)
 		)
-		(property "Manufacturer Part Number" ""
+		(property "Manufacturer Part Number" "BSZ096N10LS5ATMA1"
+			(at 218.44 93.98 0)
+			(effects
+				(font
+					(size 1.27 1.27)
+				)
+				(hide yes)
+			)
+		)
+		(property "JLCPCB Part #" ""
 			(at 218.44 93.98 0)
 			(effects
@@
 			)
 		)
-		(property "Distributor Link" ""
+		(property "Distributor Link" "https://jlcpcb.com/partdetail/3852120-IPB320P10LMATMA1/C3289219"
 			(at 172.72 88.9 0)
 			(effects
@@
 			)
 		)
-		(property "Manufacturer" ""
+		(property "Manufacturer" "Infineon Technologies"
 			(at 172.72 88.9 0)
 			(effects
@@
 			)
 		)
-		(property "Manufacturer Part Number" ""
+		(property "Manufacturer Part Number" "C3289219"
+			(at 172.72 88.9 0)
+			(effects
+				(font
+					(size 1.27 1.27)
+				)
+				(hide yes)
+			)
+		)
+		(property "JLCPCB Part #" ""
 			(at 172.72 88.9 0)
 			(effects
@@
 			)
 		)
-		(property "Distributor Link" ""
+		(property "Distributor Link" "https://jlcpcb.com/partdetail/3852120-IPB320P10LMATMA1/C3289219"
 			(at 109.22 88.9 0)
 			(effects
@@
 			)
 		)
-		(property "Manufacturer" ""
+		(property "Manufacturer" "Infineon Technologies"
 			(at 109.22 88.9 0)
 			(effects
@@
 			)
 		)
-		(property "Manufacturer Part Number" ""
+		(property "Manufacturer Part Number" "C3289219"
 			(at 109.22 88.9 0)
 			(effects
+				(font
+					(size 1.27 1.27)
+				)
+				(hide yes)
+			)
+		)
+		(property "JLCPCB Part #" ""
+			(at 109.22 88.9 0)
+			(effects

Commit message: BOM in progress v2
Parts:
- Q10, Q11, Q6, Q7: Distributor Link https://www.mouser.com/ProductDetail/Infineon-Technologies/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 -> https://jlcpcb.com/partdetail/InfineonTechnologies-BSZ096N1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; Manufacturer Part Number BSZ096N10LS5ATMA1 -> BSZ096N10LS5
Changed lines of the file:
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@@
 			)
 		)
-		(property "Distributor Link" "https://www.mouser.com/ProductDetail/Infineon-Technologies/BSZ096N10LS5ATMA1?qs=Qyx3PVvfm65D5XP%2FZXFciQ%3D%3D"
+		(property "Distributor Link" "https://jlcpcb.com/partdetail/InfineonTechnologies-BSZ096N10LS5/C534695"
 			(at 88.9 123.19 0)
 			(effects
@@
 			)
 		)
-		(property "Manufacturer Part Number" "BSZ096N10LS5ATMA1"
+		(property "Manufacturer Part Number" "BSZ096N10LS5"
 			(at 88.9 123.19 0)
 			(effects
@@
 			)
 		)
-		(property "Distributor Link" "https://www.mouser.com/ProductDetail/Infineon-Technologies/BSZ096N10LS5ATMA1?qs=Qyx3PVvfm65D5XP%2FZXFciQ%3D%3D"
+		(property "Distributor Link" "https://jlcpcb.com/partdetail/InfineonTechnologies-BSZ096N10LS5/C534695"
 			(at 62.23 93.98 0)
 			(effects
@@
 			)
 		)
-		(property "Manufacturer Part Number" "BSZ096N10LS5ATMA1"
+		(property "Manufacturer Part Number" "BSZ096N10LS5"
 			(at 62.23 93.98 0)
 			(effects
@@
 			)
 		)
-		(property "Distributor Link" "https://www.mouser.com/ProductDetail/Infineon-Technologies/BSZ096N10LS5ATMA1?qs=Qyx3PVvfm65D5XP%2FZXFciQ%3D%3D"
+		(property "Distributor Link" "https://jlcpcb.com/partdetail/InfineonTechnologies-BSZ096N10LS5/C534695"
 			(at 193.04 124.46 0)
 			(effects
@@
 			)
 		)
-		(property "Manufacturer Part Number" "BSZ096N10LS5ATMA1"
+		(property "Manufacturer Part Number" "BSZ096N10LS5"
 			(at 193.04 124.46 0)
 			(effects
@@
 			)
 		)
-		(property "Distributor Link" "https://www.mouser.com/ProductDetail/Infineon-Technologies/BSZ096N10LS5ATMA1?qs=Qyx3PVvfm65D5XP%2FZXFciQ%3D%3D"
+		(property "Distributor Link" "https://jlcpcb.com/partdetail/InfineonTechnologies-BSZ096N10LS5/C534695"
 			(at 218.44 93.98 0)
 			(effects
@@
 			)
 		)
-		(property "Manufacturer Part Number" "BSZ096N10LS5ATMA1"
+		(property "Manufacturer Part Number" "BSZ096N10LS5"
 			(at 218.44 93.98 0)
 			(effects
