File: src/bioelectric_cell_reprogramming/acdc_stimulator/kicad/pelt_cooler.kicad_sch (KiCad schematic)
At the start: 14 parts, among them J7 6620XX11122_66200211122, J8 6620XX11122_66200211122, U2 DRV8873HPWPR

Commit message: CI: footprint assignment done
Parts:
- C3: value 1uF -> 1u; footprint Capacitor_SMD:C_0201_0603Metric -> Capacitor_SMD:C_0402_1005Metric
- C4, C7: value 100nF -> 100n
- C5: value 47nF -> 47n
- C6: value 1uF -> 1u
- C8: value 10uF -> 10u; footprint Capacitor_SMD:CP_Elec_3x5.3 -> Capacitor_SMD:CP_Elec_5x5.4
- R23: value 10K -> 10k
- R24: value 1K -> 1k
- R25, R26: value 1.5K -> 1.5k

Commit message: ci: STM32 layout done and schematic annotated
Parts:
- renumbered C3 to C47, C4 to C48, C7 to C49, C5 to C50, C6 to C51, C8 to C52, J7 to J8, J8 to J9, R23 to R24, R24 to R25, R25 to R26, R26 to R27, U2 to U7
Other:
- moved on the sheet: C50, C51, J9

Commit message: fixed some more clearance errors
Parts:
- C48, C49: Distributor Link (none) -> https://jlcpcb.com/partdetail/173559-GRM155R62A104KE14D/C16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; Manufacturer (none) -> Murata Electronics; Manufacturer Part Number (none) -> GRM155R62A104KE14D

Commit message: BOM in progress
Parts:
- C47, C51: Distributor Link (none) -> https://jlcpcb.com/partdetail/30018-CL05A105KO5NNNC/C29266; Manufacturer (none) -> Samsung Electro-Mechanics; Manufacturer Part Number (none) -> CL05A105KO5NNNC
- J8, J9: Distributor Link (none) -> https://www.digikey.com/en/products/detail/w%C3%BCrth-elekt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; Manufacturer (none) -> Würth Elektronik; Manufacturer Part Number (none) -> 66200211122
- R26, R27: Distributor Link (none) -> https://jlcpcb.com/partdetail/Yageo-RC0201FR071K5L/C155737; Manufacturer (none) -> YAGEO; Manufacturer Part Number (none) -> RC0201FR-071K5L
Changed lines of the file:
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@@
+			)
+		)
+		(property "JLCPCB Part #" ""
+			(at 109.22 101.6 0)
+			(effects
+				(font
+					(size 1.27 1.27)
+				)
+				(hide yes)
 			)
 		)
@@
 			)
 		)
+		(property "JLCPCB Part #" ""
+			(at 182.88 102.87 0)
+			(effects
+				(font
+					(size 1.27 1.27)
+				)
+				(hide yes)
+			)
+		)
 		(pin "1"
 		)
@@
 			)
 		)
+		(property "JLCPCB Part #" ""
+			(at 111.76 71.12 0)
+			(effects
+				(font
+					(size 1.27 1.27)
+				)
+				(hide yes)
+			)
+		)
 		(pin "5"
 		)
@@
 			)
 		)
-		(property "Distributor Link" ""
+		(property "Distributor Link" "https://www.digikey.com/en/products/detail/w%C3%BCrth-elektronik/66200211122/4322246"
 			(at 180.34 121.92 0)
 			(effects
@@
 			)
 		)
-		(property "Manufacturer" ""
+		(property "Manufacturer" "Würth Elektronik"
 			(at 180.34 121.92 0)
 			(effects
@@
 			)
 		)
-		(property "Manufacturer Part Number" ""
+		(property "Manufacturer Part Number" "66200211122"
+			(at 180.34 121.92 0)
+			(effects
+				(font
+					(size 1.27 1.27)
+				)
+				(hide yes)
+			)
+		)
+		(property "JLCPCB Part #" ""
 			(at 180.34 121.92 0)
 			(effects
@@
 			)
 		)
-		(property "Distributor Link" ""
+		(property "Distributor Link" "https://jlcpcb.com/partdetail/Yageo-RC0201FR071K5L/C155737"
 			(at 104.14 129.54 0)
 			(effects
@@
 			)
 		)
-		(property "Manufacturer" ""
+		(property "Manufacturer" "YAGEO"
 			(at 104.14 129.54 0)
 			(effects
@@
 			)
 		)
-		(property "Manufacturer Part Number" ""
+		(property "Manufacturer Part Number" "RC0201FR-071K5L"
+			(at 104.14 129.54 0)
+			(effects
+				(font
+					(size 1.27 1.27)
+				)
+				(hide yes)
+			)
+		)
+		(property "JLCPCB Part #" ""
 			(at 104.14 129.54 0)
 			(effects
@@
 			)
 		)
+		(property "JLCPCB Part #" ""
+			(at 189.23 135.89 0)
+			(effects
+				(font
+					(size 1.27 1.27)
+				)
+				(hide yes)
+			)
+		)
 		(pin "2"
 		)
@@
 			)
 		)
+		(property "JLCPCB Part #" ""
+			(at 161.29 135.89 0)
+			(effects
+				(font
+					(size 1.27 1.27)
+				)
+				(hide yes)
+			)
+		)
 		(pin "1"
 		)
@@
 			)
 		)
-		(property "Distributor Link" ""
+		(property "Distributor Link" "https://jlcpcb.com/partdetail/Yageo-RC0201FR071K5L/C155737"
 			(at 104.14 124.46 0)
 			(effects
@@
 			)
 		)
-		(property "Manufacturer" ""
+		(property "Manufacturer" "YAGEO"
 			(at 104.14 124.46 0)
 			(effects
@@
 			)
 		)
-		(property "Manufacturer Part Number" ""
+		(property "Manufacturer Part Number" "RC0201FR-071K5L"
+			(at 104.14 124.46 0)
+			(effects
+				(font
+					(size 1.27 1.27)
+				)
+				(hide yes)
+			)
+		)
+		(property "JLCPCB Part #" ""
 			(at 104.14 124.46 0)
 			(effects
@@
 			)
 		)
-		(property "Distributor Link" ""
+		(property "Distributor Link" "https://jlcpcb.com/partdetail/30018-CL05A105KO5NNNC/C29266"
 			(at 102.87 99.06 0)
 			(effects
@@
 			)
 		)
-		(property "Manufacturer" ""
+		(property "Manufacturer" "Samsung Electro-Mechanics"
 			(at 102.87 99.06 0)
 			(effects
@@
 			)
 		)
-		(property "Manufacturer Part Number" ""
+		(property "Manufacturer Part Number" "CL05A105KO5NNNC"
+			(at 102.87 99.06 0)
+			(effects
+				(font
+					(size 1.27 1.27)
+				)
+				(hide yes)
+			)
+		)
+		(property "JLCPCB Part #" ""
 			(at 102.87 99.06 0)
 			(effects
@@
 			)
 		)
-		(property "Distributor Link" ""
+		(property "Distributor Link" "https://www.digikey.com/en/products/detail/w%C3%BCrth-elektronik/66200211122/4322246"
 			(at 157.48 66.04 0)
 			(effects
@@
 			)
 		)
-		(property "Manufacturer" ""
+		(property "Manufacturer" "Würth Elektronik"
 			(at 157.48 66.04 0)
 			(effects
@@
 			)
 		)
-		(property "Manufacturer Part Number" ""
+		(property "Manufacturer Part Number" "66200211122"
+			(at 157.48 66.04 0)
+			(effects
+				(font
+					(size 1.27 1.27)
+				)
+				(hide yes)
+			)
+		)
+		(property "JLCPCB Part #" ""
 			(at 157.48 66.04 0)
 			(effects
@@
 			)
 		)
-		(property "Distributor Link" ""
+		(property "Distributor Link" "https://jlcpcb.com/partdetail/30018-CL05A105KO5NNNC/C29266"
 			(at 182.88 111.76 0)
 			(effects
@@
 			)
 		)
-		(property "Manufacturer" ""
+		(property "Manufacturer" "Samsung Electro-Mechanics"
 			(at 182.88 111.76 0)
 			(effects
@@
 			)
 		)
-		(property "Manufacturer Part Number" ""
+		(property "Manufacturer Part Number" "CL05A105KO5NNNC"
+			(at 182.88 111.76 0)
+			(effects
+				(font
+					(size 1.27 1.27)
+				)
+				(hide yes)
+			)
+		)
+		(property "JLCPCB Part #" ""
 			(at 182.88 111.76 0)
 			(effects
@@
 			)
 		)
+		(property "JLCPCB Part #" ""
+			(at 92.71 127 0)
+			(effects
+				(font
+					(size 1.27 1.27)
+				)
+				(hide yes)
+			)
+		)
 		(pin "2"
 		)
@@
 			)
 		)
+		(property "JLCPCB Part #" ""
+			(at 175.26 135.89 0)
+			(effects
+				(font
+					(size 1.27 1.27)
+				)
+				(hide yes)
+			)
+		)
 		(pin "1"
 		)
@@
 			(at 104.14 121.92 0)
 			(effects
+				(font
+					(size 1.27 1.27)
+				)
+				(hide yes)
+			)
+		)
+		(property "JLCPCB Part #" ""
+			(at 104.14 121.92 0)
+			(effects

Commit message: fixed values for resistive divider of LDOs
Parts:
- C52: Distributor Link (none) -> https://jlcpcb.com/partdetail/Fosan-FVH050ADA100M0554/C7469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; Manufacturer (none) -> FOSAN; Manufacturer Part Number (none) -> FVH050ADA100M0554
Changed lines of the file:
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@@
 			)
 		)
-		(property "Distributor Link" ""
+		(property "Distributor Link" "https://jlcpcb.com/partdetail/Fosan-FVH050ADA100M0554/C7469956"
 			(at 189.23 135.89 0)
 			(effects
@@
 			)
 		)
-		(property "Manufacturer" ""
+		(property "Manufacturer" "FOSAN"
 			(at 189.23 135.89 0)
 			(effects
@@
 			)
 		)
-		(property "Manufacturer Part Number" ""
+		(property "Manufacturer Part Number" "FVH050ADA100M0554"
 			(at 189.23 135.89 0)
 			(effects

Commit message: ci: BOM done
Parts:
- C50: Distributor Link (none) -> https://jlcpcb.com/partdetail/MurataElectronics-GRM155R71C4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; Manufacturer (none) -> Murata Electronics; Manufacturer Part Number (none) -> GRM155R71C473KA01D
- MOSFET1: Distributor Link (none) -> https://jlcpcb.com/partdetail/InfineonTechnologies-BSZ070N0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; Manufacturer (none) -> Infineon Technologies; Manufacturer Part Number (none) -> BSZ070N08LS5
- R24: Distributor Link (none) -> https://jlcpcb.com/partdetail/Ralec-RTT01103JTH/C102690; Manufacturer (none) -> RALEC; Manufacturer Part Number (none) -> RTT01103JTH
- R25: Distributor Link (none) -> https://jlcpcb.com/partdetail/LizElec-CR0201FH1001G/C100125; Manufacturer (none) -> LIZ Elec; Manufacturer Part Number (none) -> CR0201FH1001G
- U7: Distributor Link (none) -> https://jlcpcb.com/partdetail/TexasInstruments-DRV8873HPWPR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; Manufacturer (none) -> Texas Instruments; Manufacturer Part Number (none) -> DRV8873HPWPR
Changed lines of the file:
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@@
 			)
 		)
-		(property "Distributor Link" ""
+		(property "Distributor Link" "https://jlcpcb.com/partdetail/TexasInstruments-DRV8873HPWPR/C2150604"
 			(at 109.22 101.6 0)
 			(effects
@@
 			)
 		)
-		(property "Manufacturer" ""
+		(property "Manufacturer" "Texas Instruments"
 			(at 109.22 101.6 0)
 			(effects
@@
 			)
 		)
-		(property "Manufacturer Part Number" ""
+		(property "Manufacturer Part Number" "DRV8873HPWPR"
 			(at 109.22 101.6 0)
 			(effects
@@
 			)
 		)
-		(property "Distributor Link" ""
+		(property "Distributor Link" "https://jlcpcb.com/partdetail/MurataElectronics-GRM155R71C473KA01D/C77012"
 			(at 182.88 102.87 0)
 			(effects
@@
 			)
 		)
-		(property "Manufacturer" ""
+		(property "Manufacturer" "Murata Electronics"
 			(at 182.88 102.87 0)
 			(effects
@@
 			)
 		)
-		(property "Manufacturer Part Number" ""
+		(property "Manufacturer Part Number" "GRM155R71C473KA01D"
 			(at 182.88 102.87 0)
 			(effects
@@
 			)
 		)
-		(property "Distributor Link" ""
+		(property "Distributor Link" "https://jlcpcb.com/partdetail/InfineonTechnologies-BSZ070N08LS5/C534678"
 			(at 111.76 71.12 0)
 			(effects
@@
 			)
 		)
-		(property "Manufacturer" ""
+		(property "Manufacturer" "Infineon Technologies"
 			(at 111.76 71.12 0)
 			(effects
@@
 			)
 		)
-		(property "Manufacturer Part Number" ""
+		(property "Manufacturer Part Number" "BSZ070N08LS5"
 			(at 111.76 71.12 0)
 			(effects
@@
 			)
 		)
-		(property "Distributor Link" ""
+		(property "Distributor Link" "https://jlcpcb.com/partdetail/Ralec-RTT01103JTH/C102690"
 			(at 92.71 127 0)
 			(effects
@@
 			)
 		)
-		(property "Manufacturer" ""
+		(property "Manufacturer" "RALEC"
 			(at 92.71 127 0)
 			(effects
@@
 			)
 		)
-		(property "Manufacturer Part Number" ""
+		(property "Manufacturer Part Number" "RTT01103JTH"
 			(at 92.71 127 0)
 			(effects
@@
 			)
 		)
-		(property "Distributor Link" ""
+		(property "Distributor Link" "https://jlcpcb.com/partdetail/LizElec-CR0201FH1001G/C100125"
 			(at 104.14 121.92 0)
 			(effects
@@
 			)
 		)
-		(property "Manufacturer" ""
+		(property "Manufacturer" "LIZ Elec"
 			(at 104.14 121.92 0)
 			(effects
@@
 			)
 		)
-		(property "Manufacturer Part Number" ""
+		(property "Manufacturer Part Number" "CR0201FH1001G"
 			(at 104.14 121.92 0)
 			(effects
