File: src/bioelectric_cell_reprogramming/acdc_stimulator/kicad/LTC6090_DC.kicad_sch (KiCad schematic)
At the start: 1 part, among them U4 LTC6090CFE-PBF

Commit message: CI: footprint assignment done
Parts:
- U4: footprint TSSOP-16_FE/BA_LIT -> LTC6090CFE_PBF:TSSOP-16_FE&slash_BA_LIT
Changed lines of the file:
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@@
 			)
 		)
-		(property "Footprint" "TSSOP-16_FE/BA_LIT"
+		(property "Footprint" "LTC6090CFE_PBF:TSSOP-16_FE&slash_BA_LIT"
 			(at 110.49 73.66 0)
 			(effects

Commit message: BOM in progress
Parts:
- U4: Distributor Link (none) -> https://www.digikey.com/en/products/detail/analog-devices-i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; Manufacturer (none) -> Analog Devices Inc.; Manufacturer Part Number (none) -> LTC6090CFE#PBF
Changed lines of the file:
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@@
 			)
 		)
-		(property "Distributor Link" ""
+		(property "Distributor Link" "https://www.digikey.com/en/products/detail/analog-devices-inc/LTC"
 			(at 110.49 73.66 0)
 			(effects
@@
 			)
 		)
-		(property "Manufacturer" ""
+		(property "Manufacturer" "Analog Devices Inc."
 			(at 110.49 73.66 0)
 			(effects
@@
 			)
 		)
-		(property "Manufacturer Part Number" ""
+		(property "Manufacturer Part Number" "LTC6090CFE#PBF"
 			(at 110.49 73.66 0)
 			(effects
+				(font
+					(size 1.27 1.27)
+				)
+				(hide yes)
+			)
+		)
+		(property "JLCPCB Part #" ""
+			(at 110.49 73.66 0)
+			(effects

Commit message: ci: build files for v0.0.2 generated
Parts:
- U4: Distributor Link https://www.digikey.com/en/products/detail/analog-devices-i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 -> https://www.digikey.ca/en/products/detail/analog-devices-in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
Changed lines of the file:
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@@
 			)
 		)
-		(property "Distributor Link" "https://www.digikey.com/en/products/detail/analog-devices-inc/LTC"
+		(property "Distributor Link" "https://www.digikey.ca/en/products/detail/analog-devices-inc/LTC6090CFE-PBF/3838539"
 			(at 110.49 73.66 0)
 			(effects
