File: src/bioelectric_cell_reprogramming/acdc_stimulator/kicad/acdc_stimulator.kicad_sch (KiCad schematic)
At the start: 67 parts, among them IC1 AD9833BRM-REEL7, IC2 AD5122BCPZ10-RL7, J1 Screw_Terminal_01x02, J2 Conn_ARM_SWD_TagConnect_TC203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, J3 USB_C_Receptacle_USB2.0_14P, J4 S4B-PH-SM4-TB, J5 IPL1-102-01-L-S-K, J6 Screw_Terminal_01x02, J7 IPL1-102-01-L-S-K, Q1 BSZ096N10LS5ATMA1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

Commit message: BOM in progress
Parts:
- C11, C7: footprint Capacitor_SMD:C_0402_1005Metric -> Capacitor_SMD:C_0201_0603Metric; Distributor Link (none) -> https://jlcpcb.com/partdetail/358687-GRM0335C1H300GA01D/C38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; Manufacturer (none) -> Murata Electronics; Manufacturer Part Number (none) -> GRM0335C1H300GA01D
- C16, C18: Distributor Link (none) -> https://jlcpcb.com/partdetail/6133-CL21A226MQQNNNE/C5674; Manufacturer (none) -> Samsung Electro-Mechanics; Manufacturer Part Number (none) -> CL21A226MQQNNNE
- C17, C6: Distributor Link (none) -> https://jlcpcb.com/partdetail/MurataElectronics-GRM033R61E1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; Manufacturer (none) -> Murata Electronics; Manufacturer Part Number (none) -> GRM033R61E103KA12D
- C19, C20, C5: Distributor Link (none) -> https://jlcpcb.com/partdetail/30018-CL05A105KO5NNNC/C29266; Manufacturer (none) -> Samsung Electro-Mechanics; Manufacturer Part Number (none) -> CL05A105KO5NNNC
- C21: Distributor Link (none) -> https://jlcpcb.com/partdetail/173559-GRM155R62A104KE14D/C16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; Manufacturer (none) -> Murata Electronics; Manufacturer Part Number (none) -> GRM155R62A104KE14D
- C22, C8: Distributor Link (none) -> https://jlcpcb.com/partdetail/2043-CL10A106MQ8NNNC/C1691; Manufacturer (none) -> Samsung Electro-Mechanics; Manufacturer Part Number (none) -> CL10A106MQ8NNNC
- C24, C25: value 100u -> 0; now left out of the parts list
- J1, J6: Distributor Link (none) -> https://www.mouser.com/ProductDetail/Altech/30.602-BLUE?qs=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; Manufacturer (none) -> Altech; Manufacturer Part Number (none) -> 30.602/BLUE
- J5, J7: Distributor Link (none) -> https://www.digikey.com/en/products/detail/samtec-inc/IPL1-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; Manufacturer (none) -> Samtec Inc.; Manufacturer Part Number (none) -> IPL1-102-01-L-S-K
- L1, L2, L3: value 2.5 -> 0; now left out of the parts list
- Q1: Distributor Link (none) -> https://www.mouser.com/ProductDetail/Infineon-Technologies/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; Manufacturer (none) -> Infineon Technologies; Manufacturer Part Number (none) -> BSZ096N10LS5ATMA1
- R5, R6: footprint Resistor_SMD:R_0603_1608Metric -> Resistor_SMD:R_0201_0603Metric; Distributor Link (none) -> https://jlcpcb.com/partdetail/Yageo-RC0201JR075K1L/C163490; Manufacturer (none) -> YAGEO; Manufacturer Part Number (none) -> RC0201JR-075K1L

Commit message: fixed values for resistive divider of LDOs
Parts:
- C3: Distributor Link (none) -> https://jlcpcb.com/partdetail/Fosan-FVH050ADA100M0554/C7469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; Manufacturer (none) -> FOSAN; Manufacturer Part Number (none) -> FVH050ADA100M0554
- SW1: Distributor Link (none) -> https://jlcpcb.com/partdetail/ck-KMR231GLFS/C99271; JLCPCB Part # (none) -> C99271; Manufacturer (none) -> C&K; Manufacturer Part Number (none) -> KMR231GLFS
Changed lines of the file:
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@@
 			)
 		)
-		(property "Distributor Link" ""
+		(property "Distributor Link" "https://jlcpcb.com/partdetail/Fosan-FVH050ADA100M0554/C7469956"
 			(at 26.67 36.83 0)
 			(effects
@@
 			)
 		)
-		(property "Manufacturer" ""
+		(property "Manufacturer" "FOSAN"
 			(at 26.67 36.83 0)
 			(effects
@@
 			)
 		)
-		(property "Manufacturer Part Number" ""
+		(property "Manufacturer Part Number" "FVH050ADA100M0554"
 			(at 26.67 36.83 0)
 			(effects
@@
 			)
 		)
-		(property "Distributor Link" ""
+		(property "Distributor Link" "https://jlcpcb.com/partdetail/ck-KMR231GLFS/C99271"
 			(at 49.53 186.69 0)
 			(effects
@@
 			)
 		)
-		(property "Manufacturer" ""
+		(property "Manufacturer" "C&K"
 			(at 49.53 186.69 0)
 			(effects
@@
 			)
 		)
-		(property "Manufacturer Part Number" ""
+		(property "Manufacturer Part Number" "KMR231GLFS"
 			(at 49.53 186.69 0)
 			(effects
@@
 			)
 		)
-		(property "JLCPCB Part #" ""
+		(property "JLCPCB Part #" "C99271"
 			(at 49.53 186.69 0)
 			(effects

Commit message: BOM in progress v2
Parts:
- Q1: Distributor Link https://www.mouser.com/ProductDetail/Infineon-Technologies/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 -> https://jlcpcb.com/partdetail/InfineonTechnologies-BSZ096N1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; Manufacturer Part Number BSZ096N10LS5ATMA1 -> BSZ096N10LS5
Changed lines of the file:
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@@
 			)
 		)
-		(property "Distributor Link" "https://www.mouser.com/ProductDetail/Infineon-Technologies/BSZ096N10LS5ATMA1?qs=Qyx3PVvfm65D5XP%2FZXFciQ%3D%3D"
+		(property "Distributor Link" "https://jlcpcb.com/partdetail/InfineonTechnologies-BSZ096N10LS5/C534695"
 			(at 102.87 96.52 0)
 			(effects
@@
 			)
 		)
-		(property "Manufacturer Part Number" "BSZ096N10LS5ATMA1"
+		(property "Manufacturer Part Number" "BSZ096N10LS5"
 			(at 102.87 96.52 0)
 			(effects
